File: 0128-pos-neg-boost/PCB/0128-pos-neg-boost.brd (EAGLE design)
At the start: 25.4 x 15.2 mm, 26 parts, among them U1 MIC2145

Commit message: Update C5 value
Parts:
- C5: value 10.0uF -> 10uF/16V
Changed lines of the file:
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@@
 </layers>
 <board>
-<fusionsync huburn="a.cGVyc29uYWw6dWUyYmRlZGJl" projecturn="a.cGVyc29uYWw6dWUyYmRlZGJlIzIwMTgwNTA0MTMwNTkwMzU2" f3durn="urn:adsk.wipprod:dm.lineage:kjeZz2ccQAmrtv-eR50AoA" pcbguid="5b989556-b469-4a4c-9ac9-90396e99e6a1" lastpulledtime="" lastsyncedchangeguid="" latestrevisionid="d3cb9ac3-e4af-4e66-ae5a-f31569bfd1d3" lastsyncedrevisionid="d3cb9ac3-e4af-4e66-ae5a-f31569bfd1d3" lastboardhashguid="d2c53e34-024c-a4e5-d13f-6a0aa44474a5" lastpushedtime="2022-07-11T18:14:09Z" linktopcb3d="true"/>
+<fusionsync huburn="a.cGVyc29uYWw6dWUyYmRlZGJl" projecturn="a.cGVyc29uYWw6dWUyYmRlZGJlIzIwMTgwNTA0MTMwNTkwMzU2" f3durn="urn:adsk.wipprod:dm.lineage:kjeZz2ccQAmrtv-eR50AoA" pcbguid="" lastpulledtime="" lastsyncedchangeguid="" latestrevisionid="d3cb9ac3-e4af-4e66-ae5a-f31569bfd1d3" lastsyncedrevisionid="d3cb9ac3-e4af-4e66-ae5a-f31569bfd1d3" lastboardhashguid="d2c53e34-024c-a4e5-d13f-6a0aa44474a5" lastpushedtime="2022-07-11T18:14:09Z" linktopcb3d="true"/>
 <plain>
 <wire x1="2.54" y1="0" x2="22.86" y2="0" width="0" layer="20"/>
@@
 <attribute name="VALUE" x="17.0688" y="8.7122" size="0.4064" layer="27" rot="R90" align="center"/>
 </element>
-<element name="C5" library="rlc" library_urn="urn:adsk.eagle:library:4192893" package="0603-CAP" package3d_urn="urn:adsk.eagle:package:4193021/2" value="10.0uF" x="13.462" y="3.429" smashed="yes" rot="R90">
+<element name="C5" library="rlc" library_urn="urn:adsk.eagle:library:4192893" package="0603-CAP" package3d_urn="urn:adsk.eagle:package:4193021/2" value="10uF/16V" x="13.462" y="3.429" smashed="yes" rot="R90">
 <attribute name="COST01" value="0.12" x="13.462" y="3.429" size="1.778" layer="27" rot="R90" display="off"/>
 <attribute name="COST10" value="0.09" x="13.462" y="3.429" size="1.778" layer="27" rot="R90" display="off"/>
