File: 0128-pos-neg-boost/PCB/0128-pos-neg-boost.sch (EAGLE design)
At the start: 26 parts, among them U1 MIC2145

Commit message: Update C5 value
Parts:
- C5: value 10.0uF -> 10uF/16V
Changed lines of the file:
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@@
 <part name="D2" library="diodes" library_urn="urn:adsk.eagle:library:7189447" deviceset="SCHOTTKY" device="B140" package3d_urn="urn:adsk.eagle:package:7189483/2" value="B140"/>
 <part name="D3" library="diodes" library_urn="urn:adsk.eagle:library:7189447" deviceset="SCHOTTKY" device="B140" package3d_urn="urn:adsk.eagle:package:7189483/2" value="B140"/>
-<part name="C5" library="rlc" library_urn="urn:adsk.eagle:library:4192893" deviceset="CAPACITOR" device="0603" package3d_urn="urn:adsk.eagle:package:4193021/2" value="10.0uF"/>
+<part name="C5" library="rlc" library_urn="urn:adsk.eagle:library:4192893" deviceset="CAPACITOR" device="0603" package3d_urn="urn:adsk.eagle:package:4193021/2" value="10uF/16V"/>
 <part name="SUPPLY9" library="supply" library_urn="urn:adsk.eagle:library:10485988" deviceset="GND" device=""/>
 <part name="C6" library="rlc" library_urn="urn:adsk.eagle:library:4192893" deviceset="CAPACITOR" device="0603" package3d_urn="urn:adsk.eagle:package:4193021/2" value="2.2uF"/>
