File: 0135-dcdc-neg/PCB/0135-dcdc-neg.brd (EAGLE design)
At the start: 15 x 12 mm, 13 parts

Commit message: Update Feedback Resistor value.
Parts:
- R1: value 32.2K -> 32.4K
Changed lines of the file:
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@@
 <attribute name="VALUE" x="11.646" y="6" size="0.2" layer="27" rot="R270" align="center"/>
 </element>
-<element name="R1" library="rlc" library_urn="urn:adsk.eagle:library:4192893" package="0603-RES" package3d_urn="urn:adsk.eagle:package:4193040/5" value="32.2K" x="6.3" y="4.2" smashed="yes" rot="R90">
+<element name="R1" library="rlc" library_urn="urn:adsk.eagle:library:4192893" package="0603-RES" package3d_urn="urn:adsk.eagle:package:4193040/5" value="32.4K" x="6.3" y="4.2" smashed="yes" rot="R90">
 <attribute name="COST01" value="0.10" x="6.3" y="4.2" size="1.778" layer="27" rot="R90" display="off"/>
 <attribute name="COST10" value="0.05" x="6.3" y="4.2" size="1.778" layer="27" rot="R90" display="off"/>
