File: 0135-dcdc-neg/PCB/0135-dcdc-neg.sch (EAGLE design)
At the start: 13 parts

Commit message: Update Feedback Resistor value.
Parts:
- R1: value 32.2K -> 32.4K
Changed lines of the file:
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@@
 <part name="VR1" library="regulators" library_urn="urn:adsk.eagle:library:7189770" deviceset="CUK-5P" device="-SOT-23-5" package3d_urn="urn:adsk.eagle:package:7189798/2" value="LM2611"/>
 <part name="C1" library="rlc" library_urn="urn:adsk.eagle:library:4192893" deviceset="CAPACITOR" device="0603" package3d_urn="urn:adsk.eagle:package:4193021/5" value="1uF/16V"/>
-<part name="R1" library="rlc" library_urn="urn:adsk.eagle:library:4192893" deviceset="RESISTOR" device="0603" package3d_urn="urn:adsk.eagle:package:4193040/5" value="32.2K"/>
+<part name="R1" library="rlc" library_urn="urn:adsk.eagle:library:4192893" deviceset="RESISTOR" device="0603" package3d_urn="urn:adsk.eagle:package:4193040/5" value="32.4K"/>
 <part name="D1" library="diodes" library_urn="urn:adsk.eagle:library:7189447" deviceset="SCHOTTKY" device="MBR120" package3d_urn="urn:adsk.eagle:package:7189471/3" value="MBR120"/>
 <part name="L1" library="rlc" library_urn="urn:adsk.eagle:library:4192893" deviceset="INDUCTOR" device="SMD-4.5X3.3MM" value="22uH"/>
