File: 0131-dcdc-3a/PCB-KiCAD/0131-dcdc-3a/0131-dcdc-3a.kicad_pcb (KiCad board)
At the start: 2 copper layers, 12 x 10 mm, 12 parts, among them U1 AP62300WU

Commit message: Update final parts values.
Parts:
- C2: value 0.1uF -> 10uF
- C3, C4: value 0.1uF -> 22uF
- R1: value 52.3K -> 31.6K
Changed lines of the file:
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@@
 			)
 		)
-		(property "Value" "52.3K"
+		(property "Value" "31.6K"
 			(at 0 0.2 0)
 			(layer "F.Fab")
@@
 			)
 		)
-		(property "Value" "0.1uF"
+		(property "Value" "22uF"
 			(at 0 0.2 270)
 			(layer "F.Fab")
@@
 			)
 		)
-		(property "Value" "0.1uF"
+		(property "Value" "22uF"
 			(at 0 0.2 270)
 			(layer "F.Fab")
@@
 			)
 		)
-		(property "Value" "0.1uF"
+		(property "Value" "10uF"
 			(at 0 0.2 90)
 			(layer "F.Fab")
