File: 0131-dcdc-3a/PCB-KiCAD/0131-dcdc-3a/0131-dcdc-3a.kicad_sch (KiCad schematic)
At the start: 12 parts, among them U1 AP62300WU

Commit message: Tune documentation, info block.
Other:
- company: (none) -> Circuit Monkey
- title: (none) -> #0131 DC-DC Converter, 3A
- moved on the sheet: C1, C2, C3, C4, L1, R1, R2, U1

Commit message: Fix part values in schematic.
Parts:
- C2: value 0.1uF -> 10uF
- C3, C4: value 0.1uF -> 22uF
Changed lines of the file:
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@@
 			)
 		)
-		(property "Value" "0.1uF"
+		(property "Value" "22uF"
 			(at 173.482 94.234 0)
 			(do_not_autoplace yes)
@@
 			)
 		)
-		(property "Value" "0.1uF"
+		(property "Value" "10uF"
 			(at 122.682 94.234 0)
 			(do_not_autoplace yes)
@@
 			)
 		)
-		(property "Value" "0.1uF"
+		(property "Value" "22uF"
 			(at 181.102 94.234 0)
 			(do_not_autoplace yes)

Commit message: Update final parts values.
Parts:
- R1: value 52.3K -> 31.6K
Changed lines of the file:
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@@
 			)
 		)
-		(property "Value" "52.3K"
+		(property "Value" "31.6K"
 			(at 165.1 92.71 90)
 			(do_not_autoplace yes)
