File: Synth/synth-chipz-mod-dual/synth-chipz-mod-dual.kicad_pcb (KiCad board)
At the start: 2 copper layers, 22 x 14 mm, 19 parts, among them U1 TL074

Commit message: Bump Rev to reflect PCB change.
Other:
- board text added: "Rev. B (2025/12)"
- board text removed: "Rev. A (2025/11)"
Changed lines of the file:
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@@
 	(title_block
 		(title "CHIPz - VCO/VCF Modulator")
-		(date "2025-11-05")
-		(rev "A")
+		(date "2025-12-01")
+		(rev "B")
 		(company "Circuit Monkey")
 		(comment 1 "based on a Moog design")
@@
 		)
 	)
-	(gr_text "Rev. A (2025/11)"
+	(gr_text "Rev. B (2025/12)"
 		(at 150 102.8 0)
 		(layer "B.SilkS")
